Commit message: Tuned picking for broccoli, meatball and egg

File: src/me5415_world/urdf/ur.xacro (robot description, xacro)
@@ -138,5 +138,5 @@
     </collision>
     <inertial>
-      <mass value="0.5" />
+      <mass value="0.1" />
       <origin xyz="0 0 0" rpy="0 0 0" />
       <inertia ixx="0.03" iyy="0.03" izz="0.03" ixy="0.0" ixz="0.0" iyz="0.0" />
